File: keyboards/ximi/v1/plates/ximi-plates-template.kicad_pcb (KiCad board)
At the start: 2 copper layers, 301.2 x 111.8 mm, 66 parts, among them J1 USB_C_Receptacle_USB2.0, J11 AudioJack4dpb, J2 USB_C_Receptacle_USB2.0, J7 AudioJack4dpb, SW1 SW_Push, SW10 SW_Push, SW11 SW_Push, SW12 SW_Push, SW13 SW_Push, SW14 SW_Push, SW15 SW_Push, SW16 SW_Push, SW17 SW_Push, SW18 SW_Push, SW19 SW_Push, SW2 SW_Push, SW20 SW_Push, SW21 SW_Push, SW22 SW_Push, SW23 SW_Push, SW24 SW_Push, SW25 SW_Push, SW26 SW_Push, SW27 SW_Push, SW28 SW_Push, SW29 SW_Push, SW3 SW_Push, SW30 SW_Push, SW31 SW_Push, SW32 SW_Push, SW33 SW_Push, SW34 SW_Push, SW35 SW_Push, SW36 SW_Push, SW37 SW_Push, SW38 SW_Push, SW39 SW_Push, SW4 SW_Push, SW40 SW_Push, SW41 SW_Push, SW42 SW_Push, SW47 RotaryEncoder_Switch, SW48 RotaryEncoder_Switch, SW49 SW_Push, SW5 SW_Push, SW50 SW_Push, SW6 SW_Push, SW7 SW_Push, SW8 SW_Push, SW9 SW_Push

Commit message: more progress on ximi plates, now have pointing device plates template
Parts:
- H1, H2, H3, H4, H5, H6, H7, H8: footprint MountingHole:MountingHole_2.2mm_M2_DIN965_Pad -> fingerpunch-plates:MountingHole_2.2mm_M2_DIN965_Pad
- J1, J2: footprint fingerpunch:USB_C_Receptacle_HRO_TYPE-C-31-M-12 -> fingerpunch-plates:USB_C_Receptacle_HRO_TYPE-C-31-M-12
- J11, J7: footprint Keebio-Parts:TRRS-PJ-320A -> fingerpunch-plates:TRRS-PJ-320A
